File: board/bd845-pwb.kicad_pcb (KiCad board)
At the start: 4 copper layers, 185 x 110 mm, 248 parts, among them J101 JST_VH_B4P, J301 TC2030-MCP-NL, J302 PinHeader_01x05, J401 JST_B13P_XH, J501 JST_B11P_XH_A, J601 JST_B11P_XH_A, J701 JST_B11P_XH_A, J801 JST_B11P_XH_A, J901 JST_B11P_XH_A, Q201 AOD409, Q501 AO3400A, Q601 AO3400A, Q701 AO3400A, Q801 AO3400A, Q901 AO3400A, SW101 SW_DIP_x04, U101 74HC595, U102 74HC595, U103 SRV05-4, U201 TPS54331, U202 AMS1117-3.3, U301 STM32F030C8Tx, U302 SRV05-4, U401 EL357N(C)(TA)-G, U402 EL357N(C)(TA)-G, U403 EL357N(C)(TA)-G, U404 EL357N(C)(TA)-G, U405 EL357N(C)(TA)-G, U406 SRV05-4, U407 SRV05-4, U501 SRV05-4, U601 SRV05-4, U701 SRV05-4, U801 SRV05-4, U901 SRV05-4, Y301 16Mhz

Commit message: Update PCB
Parts:
- removed TP401, TP402, TP403, TP404, TP405, TP406, TP407, TP408, TP409, TP410, TP411, TP412, TP413, TP501, TP502, TP503, TP504, TP505, TP506, TP507, TP508, TP509, TP510, TP511, TP601, TP602, TP603, TP604, TP605, TP606, TP607, TP608, TP609, TP610, TP611, TP701, TP702, TP703, TP704, TP705, TP706, TP707, TP708, TP709, TP710, TP711, TP801, TP802, TP803, TP804, TP805, TP806, TP807, TP808, TP809, TP810, TP811, TP901, TP902, TP903, TP904, TP905, TP906, TP907, TP908, TP909, TP910, TP911: TestPoint_Small, TestPoint:TestPoint_Pad_D1.0mm
- C101, C102, C103, C104: footprint Capacitor_SMD:C_0805_2012Metric -> Capacitor_SMD:C_0603_1608Metric
- J501, J601, J701, J801: footprint Connector_JST:JST_XH_B11B-XH-A_1x11_P2.50mm_Vertical -> ProjectLibrary:JST_NH_B11P-SHF-1AA_1x11_P2.50mm_Vertical
- J901: value JST_B11P_XH_A -> JST_B11P_SHF_1AA; footprint Connector_JST:JST_XH_B11B-XH-A_1x11_P2.50mm_Vertical -> ProjectLibrary:JST_NH_B11P-SHF-1AA_1x11_P2.50mm_Vertical
- moved J101 363.6 mm to (65.5, 85.3), turned to -90 degrees
- moved J302 320.1 mm to (119.9, 119.4)
- moved U302 318.7 mm to (126.1, 125.3), turned to 180 degrees
- moved J301 315.8 mm to (126.1, 129.3)
- moved R306 311.8 mm to (124.1, 120.5), turned to 90 degrees
- moved R305 309.6 mm to (126.1, 120.5), turned to 90 degrees
- moved R405 308.7 mm to (168.5, 119.5)
- moved R304 307.6 mm to (128.1, 120.5), turned to 90 degrees
- moved Y301 306.6 mm to (119.8, 102.0), turned to -90 degrees
- moved R404 304.7 mm to (173.2, 119.5)
- moved R403 300.7 mm to (178.0, 119.5)
- moved U405 300.4 mm to (168.0, 125.0), turned to -90 degrees
- moved R303 298.1 mm to (122.5, 104.5), turned to -90 degrees
- moved U404 297.2 mm to (172.8, 125.0), turned to -90 degrees
- moved R402 296.8 mm to (182.8, 119.5)
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Connections:
- R102 pad 1: Net-(U103-IO1) -> Net-(U103-IO4)
- R103 pad 1: Net-(U103-IO2) -> Net-(U103-IO3)
- R104 pad 1: Net-(U103-IO3) -> Net-(U103-IO2)
- R105 pad 1: Net-(U103-IO4) -> Net-(U103-IO1)
- R106 pad 1: Net-(U103-IO1) -> Net-(U103-IO4)
- R107 pad 1: Net-(U103-IO2) -> Net-(U103-IO3)
- R108 pad 1: Net-(U103-IO3) -> Net-(U103-IO2)
- R109 pad 1: Net-(U103-IO4) -> Net-(U103-IO1)
- SW101 pad 1: Net-(U103-IO1) -> Net-(U103-IO4)
- SW101 pad 2: Net-(U103-IO2) -> Net-(U103-IO3)
- SW101 pad 3: Net-(U103-IO3) -> Net-(U103-IO2)
- SW101 pad 4: Net-(U103-IO4) -> Net-(U103-IO1)
Routing:
- net Net-(C101-Pad2): track 5.50 -> 2.25 mm
- net GND: track 5.25 -> 4.66 mm, vias 4 -> 120
- added copper zone on B.Cu, net GND
- added copper zone on F.Cu, net GND
Other:
- board text added: "SWD"

Commit message: Update PCB
Parts:
- removed the TP201 at (497.3, 121.7)
- J401: footprint Connector_JST:JST_XH_B13B-XH-A_1x13_P2.50mm_Vertical -> ProjectLibrary:JST_NH_B13P-SHF-1AA_1x13_P2.50mm_Vertical
- moved D201 446.1 mm to (64.0, 100.8)
- moved Q201 437.7 mm to (73.8, 99.0), turned to 180 degrees
- moved C201 431.7 mm to (65.7, 92.8), turned to 180 degrees
- moved R201 424.2 mm to (77.9, 103.5), turned to 180 degrees
- moved D202 416.5 mm to (80.9, 99.0), turned to -90 degrees
- moved F201 415.9 mm to (97.0, 112.5), turned to -90 degrees
- moved C214 414.8 mm to (97.5, 117.0), turned to -90 degrees
- moved TP203 412.0 mm to (92.8, 102.8)
- moved L202 410.2 mm to (103.2, 126.5)
- moved C213 409.1 mm to (104.0, 123.5), turned to 180 degrees
- moved TP201 405.5 mm to (92.8, 97.2)
- moved TP202 405.2 mm to (92.8, 105.5)
- moved C212 404.4 mm to (100.5, 123.8), turned to 90 degrees
- moved U202 402.6 mm to (103.2, 117.0), turned to 90 degrees
- moved R209 386.3 mm to (74.8, 121.8), turned to -90 degrees
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- renumbered TP202 to TP201, TP203 to TP202, TP204 to TP203, TP205 to TP204
Connections:
- J401 pad 1: GND -> GND1
- J401 pad 10: /Comm Channel/CH3_PAD_CONN -> /Comm Channel/FL4_CONN
- J401 pad 11: /Comm Channel/CH2_PAD_CONN -> /Comm Channel/FL5_CONN
- J401 pad 12: /Comm Channel/CH1_PAD_CONN -> /Comm Channel/TEST_CONN
- J401 pad 13: GND1 -> GND
- J401 pad 2: /Comm Channel/TEST_CONN -> /Comm Channel/CH1_PAD_CONN
- J401 pad 3: /Comm Channel/FL5_CONN -> /Comm Channel/CH2_PAD_CONN
- J401 pad 4: /Comm Channel/FL4_CONN -> /Comm Channel/CH3_PAD_CONN
- J401 pad 5: /Comm Channel/FL3_CONN -> /Comm Channel/CH4_PAD_CONN
- J401 pad 6: /Comm Channel/FL2_CONN -> /Comm Channel/CH5_PAD_CONN
- J401 pad 8: /Comm Channel/CH5_PAD_CONN -> /Comm Channel/FL2_CONN
- J401 pad 9: /Comm Channel/CH4_PAD_CONN -> /Comm Channel/FL3_CONN
- U406 pad 1: /Comm Channel/FL3_CONN -> unconnected-(U406-IO1)
- U406 pad 3: /Comm Channel/FL2_CONN -> /Comm Channel/FL3_CONN
- U406 pad 6: unconnected-(U406-IO4) -> /Comm Channel/FL2_CONN
- U407 pad 1: /Comm Channel/FL3_CONN -> unconnected-(U407-IO1)
- U407 pad 3: /Comm Channel/FL2_CONN -> /Comm Channel/TEST_CONN
- U407 pad 4: /Comm Channel/FL1_CONN -> /Comm Channel/FL4_CONN
- U407 pad 6: unconnected-(U407-IO4) -> /Comm Channel/FL5_CONN
Routing:
- net /Pad Channel 5/CH_S1_CONN: track 0.00 -> 18.4 mm
- net /Pad Channel 4/CH_S1_CONN: track 0.00 -> 18.4 mm
- net /Pad Channel 3/CH_S1_CONN: track 0.00 -> 18.4 mm
- net /Pad Channel 2/CH_S4_CONN: track 0.00 -> 18.4 mm
- net /Pad Channel 2/CH_S1_CONN: track 0.00 -> 18.4 mm
- net /Pad Channel 1/CH_S4_CONN: track 0.00 -> 18.4 mm
- net /Pad Channel 1/CH_S1_CONN: track 0.00 -> 18.4 mm
- net /Pad Channel 5/CH_S4_CONN: track 0.00 -> 18.4 mm
- net /Pad Channel 3/CH_S4_CONN: track 0.00 -> 18.4 mm
- net /Pad Channel 4/CH_S4_CONN: track 0.00 -> 18.3 mm
- net /Pad Channel 5/CH_S3_CONN: track 0.00 -> 16.0 mm, vias 0 -> 2
- net /Pad Channel 5/CH_S2_CONN: track 0.00 -> 16.0 mm, vias 0 -> 2
- net /Pad Channel 4/CH_S3_CONN: track 0.00 -> 16.0 mm, vias 0 -> 2
- net /Pad Channel 4/CH_S2_CONN: track 0.00 -> 16.0 mm, vias 0 -> 2
- net /Pad Channel 3/CH_S3_CONN: track 0.00 -> 16.0 mm, vias 0 -> 2
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- added copper zone on F.Cu, net /Power/BUCK_PH
- added copper zone on F.Cu, net /Power/EXT_VCC
- added copper zone on F.Cu, net VCC
Other:
- board text added: "+12V"
- board text added: "+3V3"
- board text added: "+5V"
- board text added: "GND"
- board text added: "PAD CENTER"
- board text added: "PAD DOWN"
- board text added: "PAD LEFT"
- board text added: "PAD RIGHT"
- board text added: "PAD UP"
- board text added: "VCC"

Commit message: Update PCB
Parts:
- moved C107 2.50 mm to (178.8, 110.2)
- moved C108 2.50 mm to (177.0, 110.2)
- moved U102 2.50 mm to (185.0, 112.0)
Connections:
- U102 pad 1: /CH2_PAD -> /CH4_PAD
- U102 pad 15: /CH1_PAD -> /CH5_PAD
- U102 pad 3: /CH4_PAD -> /CH2_PAD
- U102 pad 4: /CH5_PAD -> /CH1_PAD
- U407 pad 1: unconnected-(U407-IO1) -> /Comm Channel/FL5_CONN
- U407 pad 6: /Comm Channel/FL5_CONN -> unconnected-(U407-IO4)
Routing:
- net VCC: track 0.00 -> 37.2 mm
- net /Comm Channel/CH1_PAD_CONN: track 0.00 -> 24.1 mm
- net /CH1_PAD: track 0.00 -> 22.3 mm
- net /Comm Channel/CH2_PAD_CONN: track 0.00 -> 21.8 mm
- net GND: track 11.7 -> 32.4 mm, vias 150 -> 177
- net /Comm Channel/TEST_CONN: track 0.00 -> 19.8 mm, vias 0 -> 2
- net /Comm Channel/FL1_CONN: track 0.00 -> 19.8 mm, vias 0 -> 2
- net /Comm Channel/CH3_PAD_CONN: track 0.00 -> 19.4 mm
- net /Pad Channel 5/CH_LIGHT_CONN: track 0.00 -> 19.4 mm
- net /Pad Channel 4/CH_LIGHT_CONN: track 0.00 -> 19.4 mm
- net /Pad Channel 3/CH_LIGHT_CONN: track 0.00 -> 19.4 mm
- net /Pad Channel 2/CH_LIGHT_CONN: track 0.00 -> 19.4 mm
- net /Pad Channel 1/CH_LIGHT_CONN: track 0.00 -> 19.4 mm
- net /CH2_PAD: track 0.00 -> 19.0 mm
- net /Comm Channel/CH4_PAD_CONN: track 0.00 -> 16.9 mm
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- added copper zone on F.Cu, net /Pad Channel 1/CH_LIGHT_CONN
- added copper zone on F.Cu, net /Pad Channel 2/CH_LIGHT_CONN
- added copper zone on F.Cu, net /Pad Channel 3/CH_LIGHT_CONN
- added copper zone on F.Cu, net /Pad Channel 4/CH_LIGHT_CONN
- added copper zone on F.Cu, net /Pad Channel 5/CH_LIGHT_CONN
- added copper zone on B.Cu, net GND1
- added copper zone on F.Cu, net GND1
- added copper zone on In1.Cu, net GND1
- added copper zone on In2.Cu, net GND1
Other:
- board text added: "COMM PORT"

Commit message: Update PCB
Parts:
- moved SW101 89.3 mm to (140.1, 137.5), turned to -90 degrees
- moved U103 86.7 mm to (136.2, 133.5), turned to 0 degrees
- moved R109 85.8 mm to (129.8, 128.2), turned to 90 degrees
- moved R105 83.8 mm to (131.5, 128.2), turned to 90 degrees
- moved R108 82.4 mm to (133.5, 128.2), turned to 90 degrees
- moved R104 81.1 mm to (135.2, 128.2), turned to 90 degrees
- moved R107 79.6 mm to (137.2, 128.2), turned to 90 degrees
- moved R103 78.3 mm to (139.0, 128.2), turned to 90 degrees
- moved R106 76.9 mm to (141.0, 128.2), turned to 90 degrees
- moved R102 75.8 mm to (142.8, 128.2), turned to 90 degrees
- moved C105 68.5 mm to (191.2, 87.2)
- moved C106 68.5 mm to (193.0, 87.2)
- moved U101 68.5 mm to (185.0, 85.5)
- moved C306 23.9 mm to (130.5, 92.2), turned to 0 degrees
- moved C303 18.8 mm to (145.2, 97.2), turned to 0 degrees
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Connections:
- U301 pad 10: /CH5_S1 -> /LIGHTS_SRCLK
- U301 pad 11: /CH5_S2 -> /LIGHTS_RCLK
- U301 pad 12: /CH5_S3 -> /LIGHTS_SER
- U301 pad 14: /LIGHTS_SER -> /CH5_S3
- U301 pad 15: /LIGHTS_SRCLK -> /CH5_S2
- U301 pad 16: /LIGHTS_RCLK -> /CH5_S1
- U301 pad 17: /PADS_RCLK -> /CH4_S4
- U301 pad 18: /CH1_S1 -> /CH4_S3
- U301 pad 19: /CH1_S2 -> /CH4_S2
- U301 pad 2: /OPT_COMP_MODE -> /PADS_SER
- U301 pad 20: /CH1_S3 -> /CH4_S1
- U301 pad 21: /CH3_S3 -> /CH3_S4
- U301 pad 22: /CH3_S4 -> /CH3_S3
- U301 pad 25: /CH4_S1 -> /CH3_S2
- U301 pad 26: /CH4_S2 -> /CH3_S1
- U301 pad 27: /CH4_S3 -> /CH2_S4
- U301 pad 28: /CH4_S4 -> /CH2_S3
- U301 pad 29: /PADS_SRCLK -> /CH2_S2
- U301 pad 3: /OPT_LIGHT_MODE -> /PADS_RCLK
- U301 pad 30: /PADS_SER -> /CH2_S1
- U301 pad 31: /COMM.FL1 -> /CH1_S4
- U301 pad 32: /COMM.FL2 -> /CH1_S3
- U301 pad 33: /COMM.FL3 -> /CH1_S2
- U301 pad 35: /COMM.FL5 -> /CH1_S1
- U301 pad 36: /COMM.TEST -> /OPT_LIGHT_MODE
- U301 pad 38: /COMM.FL4 -> /OPT_DEBOUNCE
- U301 pad 39: /CH1_S4 -> /OPT_COMP_MODE
- U301 pad 4: /OPT_DEBOUNCE -> /PADS_SRCLK
- U301 pad 40: /CH2_S1 -> /COMM.TEST
- U301 pad 41: /CH2_S2 -> /COMM.FL5
- U301 pad 42: /CH2_S3 -> /COMM.FL4
- U301 pad 43: /CH2_S4 -> /COMM.FL3
- U301 pad 45: /CH3_S1 -> /COMM.FL2
- U301 pad 46: /CH3_S2 -> /COMM.FL1
Routing:
- net /CH5_S4: track 0.00 -> 96.9 mm
- net /CH5_S3: track 0.00 -> 93.3 mm
- net /CH5_S2: track 0.00 -> 89.6 mm
- net /CH1_S1: track 0.00 -> 88.1 mm
- net /CH5_S1: track 0.00 -> 86.2 mm
- net /CH1_S2: track 0.00 -> 83.4 mm
- net /CH1_S3: track 0.00 -> 78.4 mm
- net /CH1_S4: track 0.00 -> 73.3 mm
- net /CH4_S4: track 0.00 -> 64.4 mm
- net /CH4_S3: track 0.00 -> 63.0 mm
- net /CH4_S2: track 0.00 -> 60.0 mm
- net /PADS_RCLK: track 0.00 -> 58.3 mm, vias 0 -> 2
- net /PADS_SRCLK: track 0.00 -> 58.0 mm
- net /CH4_S1: track 0.00 -> 57.0 mm
- net +3V3: track 11.3 -> 67.5 mm, vias 8 -> 42
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Other:
- board text added: "POWER"
- board text added: "STATUS"

Commit message: Update PCB
Parts:
- moved C302 31.0 mm to (123.8, 114.5), turned to -90 degrees
- moved R301 30.2 mm to (125.5, 114.5), turned to 90 degrees
- moved R302 29.6 mm to (127.2, 114.5), turned to -90 degrees
- moved J301 3.13 mm to (120.2, 123.2)
- moved J302 3.13 mm to (114.5, 113.4)
- moved R304 3.13 mm to (122.0, 114.5)
- moved R305 3.13 mm to (120.2, 114.5)
- moved R306 3.13 mm to (118.5, 114.5)
- moved U302 3.13 mm to (120.2, 119.2)
Connections:
- R104 pad 2: /OPT_LIGHT_MODE -> /OPT_BOOT0
- R105 pad 2: /OPT_BOOT0 -> /OPT_LIGHT_MODE
- R304 pad 1: /MCU/CONN_SWDIO -> /MCU/CONN_NRST
- R304 pad 2: /MCU/MCU_SWDIO -> /MCU/MCU_NRST
- R306 pad 1: /MCU/CONN_NRST -> /MCU/CONN_SWDIO
- R306 pad 2: /MCU/MCU_NRST -> /MCU/MCU_SWDIO
- U101 pad 1: /LIGHT_CH2 -> /LIGHT_CH5
- U101 pad 15: /LIGHT_CH1 -> /STATUS_LED_A
- U101 pad 2: /LIGHT_CH3 -> /LIGHT_CH4
- U101 pad 3: /LIGHT_CH4 -> /LIGHT_CH3
- U101 pad 4: /LIGHT_CH5 -> /LIGHT_CH2
- U101 pad 5: /STATUS_LED_A -> /LIGHT_CH1
- U302 pad 1: /MCU/CONN_SWDIO -> /MCU/CONN_NRST
- U302 pad 4: /MCU/CONN_NRST -> /MCU/CONN_SWDIO
Routing:
- net /LIGHT_CH1: track 1.75 -> 110.8 mm, vias 0 -> 2
- net /LIGHT_CH2: track 1.75 -> 83.0 mm, vias 0 -> 2
- net /LIGHTS_SER: track 0.00 -> 58.0 mm
- net /LIGHTS_RCLK: track 0.00 -> 55.8 mm
- net /LIGHTS_SRCLK: track 0.00 -> 55.7 mm, vias 0 -> 2
- net /Power/+5V: track 0.00 -> 54.6 mm, vias 0 -> 3
- net /LIGHT_CH3: track 1.75 -> 54.1 mm, vias 0 -> 2
- net /LIGHT_CH5: track 1.75 -> 48.9 mm, vias 0 -> 2
- net /STATUS_LED_A: track 0.00 -> 43.0 mm
- net /MCU/CONN_NRST: track 0.00 -> 37.8 mm, vias 0 -> 1
- net /MCU/MCU_NRST: track 0.00 -> 33.5 mm, vias 0 -> 2
- net /MCU/MCU_SWDIO: track 0.00 -> 23.1 mm, vias 0 -> 2
- net /LIGHT_CH4: track 1.75 -> 24.2 mm, vias 0 -> 2
- net /MCU/CONN_SWCLK: track 0.00 -> 20.3 mm, vias 0 -> 1
- net /COMM.TEST: track 26.6 -> 45.9 mm
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- added copper zone on F.Cu, net +3V3
- added copper zone on F.Cu, net /Power/+5V
- added copper zone on F.Cu, net /Power/LDO_VI
- added copper zone on F.Cu, net /Power/LDO_VO
- added copper zone on B.Cu, net VCC
