File: board/bd845-pwb.kicad_sch (KiCad schematic)
At the start: 8 parts

Commit message: Update schematic
Parts:
- added C105, C108: 10n, symbol Device:C_Small
- added C106, C107: 100n, symbol Device:C_Small
- added D101: Status, symbol Device:LED_Small
- added J101: JST_VH_B4P, symbol Connector_Generic:Conn_01x04
- added R101: 1k, symbol Device:R_Small
- added R? (x4): 150R, symbol Device:R_Small
- added R? (x4): 10k, symbol Device:R_Small
- added SW101: SW_DIP_x04, symbol Switch:SW_DIP_x04
- added U101, U102: 74HC595, symbol 74xx:74HC595
- added U?: SRV05-4, Package_TO_SOT_SMD:SOT-23-6, symbol ProjectLibrary:SRV05-4
- renumbered C1 to C101, C2 to C102, C3 to C103, C401 to C104, H1 to H101, H2 to H102, H3 to H103, H4 to H104
Connections:
- net GND: now also C105.2, C106.2, C107.2, C108.2, J101.3 (Pin_3), J101.4 (Pin_4), R101.2, R?.2, R?.2, R?.2, R?.2, U101.13 (~{OE}), U101.8 (GND), U102.13 (~{OE}), U102.8 (GND), U?.2 (VN)
- new net: R?.1, R?.1, SW101.4, U?.6 (IO4)
- new net: R?.1, R?.1, SW101.2, U?.3 (IO2)
- new net: R?.1, R?.1, SW101.1, U?.1 (IO1)
- new net: R?.1, R?.1, SW101.3, U?.4 (IO3)
- new net +3V3: C105.1, C106.1, C107.1, C108.1, SW101.5, SW101.6, SW101.7, SW101.8, U101.10 (~{SRCLR}), U101.16 (VCC), U102.10 (~{SRCLR}), U102.16 (VCC), U?.5 (VP)
- new net CH1_PAD: U102.15 (QA)
- new net CH2_PAD: U102.1 (QB)
- new net CH3_PAD: U102.2 (QC)
- new net CH4_PAD: U102.3 (QD)
- new net CH5_PAD: U102.4 (QE)
- new net LIGHTS_RCLK: U101.12 (RCLK)
- new net LIGHTS_SER: U101.14 (SER)
- new net LIGHTS_SRCLK: U101.11 (SRCLK)
- new net LIGHT_CH1: U101.15 (QA)
- new net LIGHT_CH2: U101.1 (QB)
- new net LIGHT_CH3: U101.2 (QC)
- new net LIGHT_CH4: U101.3 (QD)
- new net LIGHT_CH5: U101.4 (QE)
- new net OPT_BOOT0: R?.2
- new net OPT_COMP_MODE: R?.2
- new net OPT_DEBOUNCE: R?.2
- new net OPT_LIGHT_MODE: R?.2
- new net PADS_RCLK: U102.12 (RCLK)
- new net PADS_SER: U102.14 (SER)
- new net PADS_SRCLK: U102.11 (SRCLK)
- new net Power/EXT_VCC: J101.1 (Pin_1), J101.2 (Pin_2)
- new net STATUS_LED_A: D101.2 (A), U101.5 (QF)
- new net STATUS_LED_K: D101.1 (K), R101.1
- no-connect marks 0 -> 8
Other:
- added sheet Comm Channel (comm_channel.kicad_sch)
- added sheet Pad Channel 1 (pad_channel.kicad_sch)
- added sheet Pad Channel 2 (pad_channel.kicad_sch)
- added sheet Pad Channel 3 (pad_channel.kicad_sch)
- added sheet Pad Channel 4 (pad_channel.kicad_sch)
- added sheet Pad Channel 5 (pad_channel.kicad_sch)
- sheet MCU ports: added CH1_S1, CH1_S2, CH1_S3, CH1_S4, CH2_S1, CH2_S2, CH2_S3, CH2_S4, CH3_S1, CH3_S2, CH3_S3, CH3_S4, CH4_S1, CH4_S2, CH4_S3, CH4_S4, CH5_S1, CH5_S2, CH5_S3, CH5_S4, FL1, FL2, FL3, FL4, FL5, LIGHTS_RCLK, LIGHTS_SER, LIGHTS_SRCLK, OPT_BOOT0, OPT_DEBOUNCE, OPT_LIGHT_MODE, OPT_SENSOR_MODE, PADS_RCLK, PADS_SER, PADS_SRCLK, TEST; removed none
- sheet Power ports: added +3V3, +5V, EXT_VCC, VCC; removed none
- note added: "CH1_S[1..4]"
- note added: "CH2_S[1..4]"
- note added: "CH3_S[1..4]"
- note added: "CH4_S[1..4]"
- note added: "CH5_S[1..4]"
- note added: "COMM{FL[1..5] TEST}"
- note added: "ESD protection. Series resistors limit maximum short-circuit current."
- note added: "LIGHT_CH[1..5]"
- note added: "Options"
- note added: "Root page"
- note added: "Status Indicators"
- company: (none) -> BlueDot, Vincenzo Fortunato
- title: (none) -> BD845-PWB
- moved on the sheet: C101, C102, C103, C104, H101, H102, H103, H104

Commit message: Schematic done
Parts:
- C101, C102, C103, C104: footprint (none) -> Capacitor_SMD:C_0805_2012Metric
- C105, C106, C107, C108: footprint (none) -> Capacitor_SMD:C_0603_1608Metric
- D101: footprint (none) -> LED_SMD:LED_0805_2012Metric
- H101, H102, H103, H104: footprint (none) -> MountingHole:MountingHole_4mm_Pad_Via
- J101: footprint (none) -> Connector_JST:JST_VH_B4P-VH_1x04_P3.96mm_Vertical
- R101, R? (x8): footprint (none) -> Resistor_SMD:R_0603_1608Metric
- SW101: footprint (none) -> Button_Switch_THT:SW_DIP_SPSTx04_Slide_9.78x12.34mm_W7.62mm_P2.54mm
- U101, U102: footprint (none) -> Package_SO:SO-16_3.9x9.9mm_P1.27mm
Other:
- note added: "Status Indicator"
- note removed: "CH1_S[1..4]"
- note removed: "CH2_S[1..4]"
- note removed: "CH3_S[1..4]"
- note removed: "CH4_S[1..4]"
- note removed: "CH5_S[1..4]"
- note removed: "COMM{FL[1..5] TEST}"
- note removed: "LIGHT_CH[1..5]"
- note removed: "Status Indicators"
- moved on the sheet: C101, C102, C103, C104, C105, C106, C107, C108, D101, H101, H102, H103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

Commit message: Update PCB
Parts:
- C101, C102, C103, C104: footprint Capacitor_SMD:C_0805_2012Metric -> Capacitor_SMD:C_0603_1608Metric
Connections:
- net at R?.1, R?.1, SW101.4: now also U?.1 (IO1); no longer U?.6 (IO4)
- net at R?.1, R?.1, SW101.2: now also U?.4 (IO3); no longer U?.3 (IO2)
- net at R?.1, R?.1, SW101.1: now also U?.6 (IO4); no longer U?.1 (IO1)
- net at R?.1, R?.1, SW101.3: now also U?.3 (IO2); no longer U?.4 (IO3)
Changed lines of the file:
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@@
     (company "BlueDot, Vincenzo Fortunato")
   )
-  (junction (at 252.73 127) (diameter 0) (color 0 0 0 0)
-  )
   (junction (at 86.36 162.56) (diameter 0) (color 0 0 0 0)
   )
   (junction (at 224.79 137.16) (diameter 0) (color 0 0 0 0)
   )
+  (junction (at 245.11 129.54) (diameter 0) (color 0 0 0 0)
+  )
   (junction (at 234.95 137.16) (diameter 0) (color 0 0 0 0)
   )
   (junction (at 229.87 124.46) (diameter 0) (color 0 0 0 0)
   )
+  (junction (at 248.92 127) (diameter 0) (color 0 0 0 0)
+  )
   (junction (at 224.79 121.92) (diameter 0) (color 0 0 0 0)
   )
@@
   (junction (at 96.52 93.98) (diameter 0) (color 0 0 0 0)
   )
-  (junction (at 256.54 129.54) (diameter 0) (color 0 0 0 0)
+  (junction (at 256.54 121.92) (diameter 0) (color 0 0 0 0)
   )
   (junction (at 229.87 137.16) (diameter 0) (color 0 0 0 0)
   )
-  (junction (at 248.92 124.46) (diameter 0) (color 0 0 0 0)
-  )
-  (junction (at 245.11 121.92) (diameter 0) (color 0 0 0 0)
-  )
   (junction (at 133.35 181.61) (diameter 0) (color 0 0 0 0)
+  )
+  (junction (at 252.73 124.46) (diameter 0) (color 0 0 0 0)
   )
   (junction (at 229.87 52.07) (diameter 0) (color 0 0 0 0)
@@
     (stroke (width 0) (type default))
   )
-  (wire (pts (xy 229.87 124.46) (xy 248.92 124.46))
+  (wire (pts (xy 229.87 124.46) (xy 252.73 124.46))
     (stroke (width 0) (type default))
   )
@@
     (stroke (width 0) (type default))
   )
+  (wire (pts (xy 252.73 124.46) (xy 259.08 124.46))
+    (stroke (width 0) (type default))
+  )
   (bus (pts (xy 132.08 76.2) (xy 132.08 73.66))
     (stroke (width 0) (type default))
@@
     (stroke (width 0) (type default))
   )
-  (wire (pts (xy 245.11 121.92) (xy 259.08 121.92))
-    (stroke (width 0) (type default))
-  )
   (wire (pts (xy 185.42 72.39) (xy 201.93 72.39))
     (stroke (width 0) (type default))
@@
     (stroke (width 0) (type default))
   )
+  (wire (pts (xy 256.54 121.92) (xy 259.08 121.92))
+    (stroke (width 0) (type default))
+  )
   (bus (pts (xy 60.96 52.07) (xy 60.96 54.61))
     (stroke (width 0) (type default))
@@
     (stroke (width 0) (type default))
   )
+  (wire (pts (xy 248.92 127) (xy 248.92 139.7))
+    (stroke (width 0) (type default))
+  )
   (wire (pts (xy 185.42 74.93) (xy 209.55 74.93))
     (stroke (width 0) (type default))
@@
     (stroke (width 0) (type default))
   )
-  (wire (pts (xy 256.54 129.54) (xy 256.54 139.7))
-    (stroke (width 0) (type default))
-  )
   (wire (pts (xy 185.42 41.91) (xy 196.85 41.91))
     (stroke (width 0) (type default))
@@
   )
   (wire (pts (xy 274.32 121.92) (xy 276.86 121.92))
-    (stroke (width 0) (type default))
-  )
-  (wire (pts (xy 248.92 124.46) (xy 248.92 139.7))
     (stroke (width 0) (type default))
   )
@@
     (stroke (width 0) (type default))
   )
+  (wire (pts (xy 245.11 129.54) (xy 259.08 129.54))
+    (stroke (width 0) (type default))
+  )
   (polyline (pts (xy 171.45 152.4) (xy 171.45 138.43))
     (stroke (width 0) (type default))
@@
     (stroke (width 0) (type default))
   )
+  (wire (pts (xy 248.92 127) (xy 259.08 127))
+    (stroke (width 0) (type default))
+  )
   (wire (pts (xy 207.01 77.47) (xy 207.01 67.31))
     (stroke (width 0) (type default))
@@
     (stroke (width 0) (type default))
   )
+  (wire (pts (xy 245.11 129.54) (xy 245.11 139.7))
+    (stroke (width 0) (type default))
+  )
   (wire (pts (xy 219.71 52.07) (xy 229.87 52.07))
     (stroke (width 0) (type default))
@@
     (stroke (width 0) (type default))
   )
-  (wire (pts (xy 248.92 124.46) (xy 259.08 124.46))
-    (stroke (width 0) (type default))
-  )
-  (wire (pts (xy 245.11 121.92) (xy 245.11 139.7))
-    (stroke (width 0) (type default))
-  )
   (bus (pts (xy 199.39 41.91) (xy 199.39 39.37))
     (stroke (width 0) (type default))
@@
     (stroke (width 0) (type default))
   )
-  (wire (pts (xy 224.79 121.92) (xy 245.11 121.92))
+  (wire (pts (xy 224.79 121.92) (xy 256.54 121.92))
     (stroke (width 0) (type default))
   )
@@
     (stroke (width 0) (type default))
   )
+  (wire (pts (xy 256.54 121.92) (xy 256.54 139.7))
+    (stroke (width 0) (type default))
+  )
   (wire (pts (xy 96.52 168.91) (xy 97.79 168.91))
     (stroke (width 0) (type default))
@@
     (stroke (width 0) (type default))
   )
-  (wire (pts (xy 240.03 129.54) (xy 256.54 129.54))
+  (wire (pts (xy 240.03 129.54) (xy 245.11 129.54))
     (stroke (width 0) (type default))
   )
@@
     (stroke (width 0) (type default))
   )
-  (wire (pts (xy 234.95 127) (xy 252.73 127))
-    (stroke (width 0) (type default))
-  )
   (wire (pts (xy 142.24 44.45) (xy 151.13 44.45))
     (stroke (width 0) (type default))
@@
     (stroke (width 0) (type default))
   )
-  (wire (pts (xy 256.54 129.54) (xy 259.08 129.54))
-    (stroke (width 0) (type default))
-  )
   (wire (pts (xy 133.35 181.61) (xy 133.35 184.15))
     (stroke (width 0) (type default))
   )
-  (wire (pts (xy 252.73 127) (xy 252.73 139.7))
-    (stroke (width 0) (type default))
-  )
-  (wire (pts (xy 252.73 127) (xy 259.08 127))
+  (wire (pts (xy 234.95 127) (xy 248.92 127))
     (stroke (width 0) (type default))
   )
@@
   )
   (bus (pts (xy 68.58 27.94) (xy 68.58 135.89))
+    (stroke (width 0) (type default))
+  )
+  (wire (pts (xy 252.73 124.46) (xy 252.73 139.7))
     (stroke (width 0) (type default))
   )
@@
       (effects (font (size 1.27 1.27)))
     )
-    (property "Footprint" "Capacitor_SMD:C_0805_2012Metric" (at 93.98 168.91 0)
+    (property "Footprint" "Capacitor_SMD:C_0603_1608Metric" (at 93.98 168.91 0)
       (effects (font (size 1.27 1.27)) hide)
     )
@@
       (project "bd845-pwb"
         (path "/c0443f53-6229-4858-b0f1-180b8ed8e6c2"
-          (reference "C103") (unit 1) (value "1n") (footprint "Capacitor_SMD:C_0805_2012Metric")
+          (reference "C103") (unit 1) (value "1n") (footprint "Capacitor_SMD:C_0603_1608Metric")
         )
       )
@@
       (effects (font (size 1.27 1.27)))
     )
-    (property "Footprint" "Capacitor_SMD:C_0805_2012Metric" (at 93.98 175.26 0)
+    (property "Footprint" "Capacitor_SMD:C_0603_1608Metric" (at 93.98 175.26 0)
       (effects (font (size 1.27 1.27)) hide)
     )
@@
       (project "bd845-pwb"
         (path "/c0443f53-6229-4858-b0f1-180b8ed8e6c2"
-          (reference "C104") (unit 1) (value "1n") (footprint "Capacitor_SMD:C_0805_2012Metric")
+          (reference "C104") (unit 1) (value "1n") (footprint "Capacitor_SMD:C_0603_1608Metric")
         )
       )
@@
       (effects (font (size 1.27 1.27)))
     )
-    (property "Footprint" "Capacitor_SMD:C_0805_2012Metric" (at 93.98 162.56 0)
+    (property "Footprint" "Capacitor_SMD:C_0603_1608Metric" (at 93.98 162.56 0)
       (effects (font (size 1.27 1.27)) hide)
     )
@@
       (project "bd845-pwb"
         (path "/c0443f53-6229-4858-b0f1-180b8ed8e6c2"
-          (reference "C102") (unit 1) (value "1n") (footprint "Capacitor_SMD:C_0805_2012Metric")
+          (reference "C102") (unit 1) (value "1n") (footprint "Capacitor_SMD:C_0603_1608Metric")
         )
       )
@@
       (effects (font (size 1.27 1.27)))
     )
-    (property "Footprint" "Capacitor_SMD:C_0805_2012Metric" (at 93.98 156.21 0)
+    (property "Footprint" "Capacitor_SMD:C_0603_1608Metric" (at 93.98 156.21 0)
       (effects (font (size 1.27 1.27)) hide)
     )
@@
       (project "bd845-pwb"
         (path "/c0443f53-6229-4858-b0f1-180b8ed8e6c2"
-          (reference "C101") (unit 1) (value "1n") (footprint "Capacitor_SMD:C_0805_2012Metric")
-        )
-      )
+          (reference "C101") (unit 1) (value "1n") (footprint "Capacitor_SMD:C_0603_1608Metric")
+        )
+      )

Commit message: Update PCB
Connections:
- net CH1_PAD: now also U102.4 (QE); no longer U102.15 (QA)
- net CH2_PAD: now also U102.3 (QD); no longer U102.1 (QB)
- net CH4_PAD: now also U102.1 (QB); no longer U102.3 (QD)
- net CH5_PAD: now also U102.15 (QA); no longer U102.4 (QE)
Changed lines of the file:
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@@
+    (stroke (width 0) (type default))
+  )
+  (wire (pts (xy 229.87 69.85) (xy 251.46 69.85))
     (stroke (width 0) (type default))
   )
@@
   )
   (wire (pts (xy 144.78 143.51) (xy 160.02 143.51))
-    (stroke (width 0) (type default))
-  )
-  (wire (pts (xy 229.87 72.39) (xy 251.46 72.39))
     (stroke (width 0) (type default))
   )
@@
     (stroke (width 0) (type default))
   )
+  (wire (pts (xy 229.87 74.93) (xy 251.46 74.93))
+    (stroke (width 0) (type default))
+  )
   (wire (pts (xy 224.79 121.92) (xy 256.54 121.92))
     (stroke (width 0) (type default))
@@
     (stroke (width 0) (type default))
   )
+  (wire (pts (xy 229.87 80.01) (xy 251.46 80.01))
+    (stroke (width 0) (type default))
+  )
   (wire (pts (xy 185.42 34.29) (xy 196.85 34.29))
     (stroke (width 0) (type default))
@@
     (stroke (width 0) (type default))
   )
+  (bus (pts (xy 129.54 92.71) (xy 129.54 90.17))
+    (stroke (width 0) (type default))
+  )
+  (wire (pts (xy 234.95 137.16) (xy 234.95 135.89))
+    (stroke (width 0) (type default))
+  )
+  (wire (pts (xy 86.36 162.56) (xy 86.36 156.21))
+    (stroke (width 0) (type default))
+  )
+  (wire (pts (xy 86.36 156.21) (xy 91.44 156.21))
+    (stroke (width 0) (type default))
+  )
   (wire (pts (xy 229.87 77.47) (xy 251.46 77.47))
     (stroke (width 0) (type default))
   )
-  (bus (pts (xy 129.54 92.71) (xy 129.54 90.17))
-    (stroke (width 0) (type default))
-  )
-  (wire (pts (xy 234.95 137.16) (xy 234.95 135.89))
-    (stroke (width 0) (type default))
-  )
-  (wire (pts (xy 86.36 162.56) (xy 86.36 156.21))
-    (stroke (width 0) (type default))
-  )
-  (wire (pts (xy 86.36 156.21) (xy 91.44 156.21))
-    (stroke (width 0) (type default))
-  )
   (wire (pts (xy 49.53 90.17) (xy 60.96 90.17))
     (stroke (width 0) (type default))
@@
     (stroke (width 0) (type default))
   )
-  (wire (pts (xy 229.87 80.01) (xy 251.46 80.01))
-    (stroke (width 0) (type default))
-  )
   (bus (pts (xy 134.62 62.23) (xy 134.62 64.77))
     (stroke (width 0) (type default))
@@
     (stroke (width 0) (type default))
   )
+  (wire (pts (xy 229.87 72.39) (xy 251.46 72.39))
+    (stroke (width 0) (type default))
+  )
   (wire (pts (xy 185.42 127) (xy 209.55 127))
     (stroke (width 0) (type default))
@@
     (stroke (width 0) (type default))
   )
-  (wire (pts (xy 229.87 69.85) (xy 251.46 69.85))
-    (stroke (width 0) (type default))
-  )
   (bus (pts (xy 63.5 22.86) (xy 63.5 80.01))
     (stroke (width 0) (type default))
@@
   )
   (wire (pts (xy 224.79 137.16) (xy 229.87 137.16))
-    (stroke (width 0) (type default))
-  )
-  (wire (pts (xy 229.87 74.93) (xy 251.46 74.93))
     (stroke (width 0) (type default))
   )
@@
     (effects (font (size 1.27 1.27)) (justify left bottom))
   )
+  (label "CH3_PAD" (at 231.14 74.93 0) (fields_autoplaced)
+    (effects (font (size 1.27 1.27)) (justify left bottom))
+  )
   (label "LIGHT_CH5" (at 91.44 114.3 0) (fields_autoplaced)
     (effects (font (size 1.27 1.27)) (justify left bottom))
@@
     (effects (font (size 1.27 1.27)) (justify left bottom))
   )
+  (label "CH2_PAD" (at 231.14 77.47 0) (fields_autoplaced)
+    (effects (font (size 1.27 1.27)) (justify left bottom))
+  )
   (label "CH1_S[1..4]" (at 74.93 20.32 0) (fields_autoplaced)
     (effects (font (size 1.27 1.27)) (justify left bottom))
@@
     (effects (font (size 1.27 1.27)) (justify left bottom))
   )
-  (label "CH2_PAD" (at 231.1365 72.39 0) (fields_autoplaced)
-    (effects (font (size 1.27 1.27)) (justify left bottom))
-  )
   (label "STATUS_LED_K" (at 146.05 143.51 0) (fields_autoplaced)
     (effects (font (size 1.27 1.27)) (justify left bottom))
   )
   (label "CH5_S3" (at 50.8 171.45 0) (fields_autoplaced)
-    (effects (font (size 1.27 1.27)) (justify left bottom))
-  )
-  (label "CH5_PAD" (at 231.1365 80.01 0) (fields_autoplaced)
     (effects (font (size 1.27 1.27)) (justify left bottom))
   )
@@
     (effects (font (size 1.27 1.27)) (justify left bottom))
   )
-  (label "CH3_PAD" (at 231.1365 74.93 0) (fields_autoplaced)
-    (effects (font (size 1.27 1.27)) (justify left bottom))
-  )
   (label "CH4_S1" (at 50.8 138.43 0) (fields_autoplaced)
     (effects (font (size 1.27 1.27)) (justify left bottom))
@@
     (effects (font (size 1.27 1.27)) (justify left bottom))
   )
+  (label "CH4_PAD" (at 231.14 72.39 0) (fields_autoplaced)
+    (effects (font (size 1.27 1.27)) (justify left bottom))
+  )
   (label "COMM.FL5" (at 186.69 41.91 0) (fields_autoplaced)
     (effects (font (size 1.27 1.27)) (justify left bottom))
   )
-  (label "CH4_PAD" (at 231.1365 77.47 0) (fields_autoplaced)
-    (effects (font (size 1.27 1.27)) (justify left bottom))
-  )
   (label "CH4_S[1..4]" (at 74.93 27.94 0) (fields_autoplaced)
     (effects (font (size 1.27 1.27)) (justify left bottom))
@@
     (effects (font (size 1.27 1.27)) (justify left bottom))
   )
-  (label "CH1_PAD" (at 231.1365 69.85 0) (fields_autoplaced)
-    (effects (font (size 1.27 1.27)) (justify left bottom))
-  )
   (label "CH3_S[1..4]" (at 74.93 25.4 0) (fields_autoplaced)
     (effects (font (size 1.27 1.27)) (justify left bottom))
   )
   (label "OPT_DEBOUNCE" (at 193.04 124.46 0) (fields_autoplaced)
+    (effects (font (size 1.27 1.27)) (justify left bottom))
+  )
+  (label "CH1_PAD" (at 231.14 80.01 0) (fields_autoplaced)
     (effects (font (size 1.27 1.27)) (justify left bottom))
   )
@@
   )
   (label "CH3_S3" (at 142.24 69.85 0) (fields_autoplaced)
+    (effects (font (size 1.27 1.27)) (justify left bottom))
+  )
+  (label "CH5_PAD" (at 231.14 69.85 0) (fields_autoplaced)
     (effects (font (size 1.27 1.27)) (justify left bottom))
   )
@@
       (effects (font (size 1.27 1.27)) (justify left))
     )
-    (pin "CH5_PAD" input (at 251.46 80.01 180)
+    (pin "CH5_PAD" input (at 251.46 69.85 180)
       (effects (font (size 1.27 1.27)) (justify left))
     )
-    (pin "CH4_PAD" input (at 251.46 77.47 180)
+    (pin "CH4_PAD" input (at 251.46 72.39 180)
       (effects (font (size 1.27 1.27)) (justify left))
     )
-    (pin "CH2_PAD" input (at 251.46 72.39 180)
+    (pin "CH2_PAD" input (at 251.46 77.47 180)
       (effects (font (size 1.27 1.27)) (justify left))
     )
-    (pin "CH1_PAD" input (at 251.46 69.85 180)
+    (pin "CH1_PAD" input (at 251.46 80.01 180)
       (effects (font (size 1.27 1.27)) (justify left))
     )

Commit message: Update PCB
Parts:
- R101: value 1k -> 330R
Connections:
- net LIGHT_CH1: now also U101.5 (QF); no longer U101.15 (QA)
- net LIGHT_CH2: now also U101.4 (QE); no longer U101.1 (QB)
- net LIGHT_CH3: now also U101.3 (QD); no longer U101.2 (QC)
- net LIGHT_CH4: now also U101.2 (QC); no longer U101.3 (QD)
- net LIGHT_CH5: now also U101.1 (QB); no longer U101.4 (QE)
- net OPT_BOOT0: now also R?.2; no longer R?.2
- net OPT_LIGHT_MODE: now also R?.2; no longer R?.2
- net STATUS_LED_A: now also U101.15 (QA); no longer U101.5 (QF)

Commit message: Update PCB
Connections:
- net +3V3: now also SW101.1, SW101.2, SW101.3, SW101.4; no longer SW101.5, SW101.6, SW101.7, SW101.8
- net OPT_LIGHT_SW: now reaches R?.1, R?.1, U?.1 (IO1)
- net OPT_LIGHT_SW: now also SW101.8; no longer SW101.4
- net OPT_DEBOUNCE_SW: now reaches R?.1, R?.1, U?.4 (IO3)
- net OPT_DEBOUNCE_SW: now also SW101.6; no longer SW101.2
- net OPT_LEGACY_SW: now reaches R?.1, R?.1, U?.6 (IO4)
- net OPT_LEGACY_SW: now also SW101.5; no longer SW101.1
- net OPT_BOOT0_SW: now reaches R?.1, R?.1, U?.3 (IO2)
- net OPT_BOOT0_SW: now also SW101.7; no longer SW101.3
- net OPT_COMP_MODE renamed OPT_LEGACY
- net OPT_LIGHT_MODE renamed OPT_LIGHT
Other:
- sheet MCU ports: added OPT_LEGACY, OPT_LIGHT; removed OPT_LIGHT_MODE, OPT_SENSOR_MODE
- moved on the sheet: SW101

Commit message: Select input TVS diode
Other:
- title: BD845-PWB -> BD845-PWB SCH
Changed lines of the file:
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@@
   (paper "A4")
   (title_block
-    (title "BD845-PWB")
+    (title "BD845-PWB SCH")
     (date "2022-11-27")
-    (rev "1")
+    (rev "1.0.0")
     (company "BlueDot, Vincenzo Fortunato")
   )
