File: board/comm_channel.kicad_sch (KiCad schematic)
At the start: 25 parts, among them J401 JST_B13P_XH, U401 EL357N(C)(TA)-G, U402 EL357N(C)(TA)-G, U403 EL357N(C)(TA)-G, U404 EL357N(C)(TA)-G, U405 EL357N(C)(TA)-G

Commit message: Schematic done
Parts:
- added TP401, TP402, TP403, TP404, TP405, TP406, TP407, TP408, TP409, TP410, TP411, TP412, TP413: TestPoint_Small, TestPoint:TestPoint_Pad_D1.0mm, symbol Connector:TestPoint_Small
- J401: footprint (none) -> Connector_JST:JST_XH_B13B-XH-A_1x13_P2.50mm_Vertical
- R401, R402, R403, R404, R405, R412, R413, R414, R415, R416, R417, R? (x6): footprint (none) -> Resistor_SMD:R_0603_1608Metric
Connections:
- net CH1_PAD_CONN: now also TP412.1
- net CH2_PAD_CONN: now also TP411.1
- net CH3_PAD_CONN: now also TP410.1
- net CH4_PAD_CONN: now also TP409.1
- net CH5_PAD_CONN: now also TP408.1
- net FL1_CONN: now also R412.1, R?.1, U?.4 (IO3), U?.4 (IO3), TP407.1
- net FL2_CONN: now also TP406.1; no longer R412.1, R?.1, U?.4 (IO3), U?.4 (IO3)
- net FL3_CONN: now also TP405.1
- net FL4_CONN: now also TP404.1
- net FL5_CONN: now also TP403.1
- net GND: now also TP401.1
- net GND1: now also TP413.1
- net TEST_CONN: now also TP402.1

Commit message: Update PCB
Parts:
- removed TP401, TP402, TP403, TP404, TP405, TP406, TP407, TP408, TP409, TP410, TP411, TP412, TP413: TestPoint_Small, TestPoint:TestPoint_Pad_D1.0mm, symbol Connector:TestPoint_Small
Other:
- moved on the sheet: J401

Commit message: Update PCB
Parts:
- J401: footprint Connector_JST:JST_XH_B13B-XH-A_1x13_P2.50mm_Vertical -> ProjectLibrary:JST_NH_B13P-SHF-1AA_1x13_P2.50mm_Vertical
Connections:
- net CH1_PAD_CONN: now also J401.2 (Pin_2); no longer J401.12 (Pin_12)
- net CH2_PAD_CONN: now also J401.3 (Pin_3); no longer J401.11 (Pin_11)
- net CH3_PAD_CONN: now also J401.4 (Pin_4); no longer J401.10 (Pin_10)
- net CH4_PAD_CONN: now also J401.5 (Pin_5); no longer J401.9 (Pin_9)
- net CH5_PAD_CONN: now also J401.6 (Pin_6); no longer J401.8 (Pin_8)
- net FL1_CONN: no longer U?.4 (IO3)
- net FL2_CONN: now also J401.8 (Pin_8), U?.6 (IO4); no longer J401.6 (Pin_6), U?.3 (IO2), U?.3 (IO2)
- net FL3_CONN: now also J401.9 (Pin_9), U?.3 (IO2); no longer J401.5 (Pin_5), U?.1 (IO1), U?.1 (IO1)
- net FL4_CONN: now also J401.10 (Pin_10), U?.4 (IO3); no longer J401.4 (Pin_4)
- net FL5_CONN: now also J401.11 (Pin_11), U?.6 (IO4); no longer J401.3 (Pin_3)
- net GND: now also J401.13 (Pin_13); no longer J401.1 (Pin_1)
- net GND1: now also J401.1 (Pin_1); no longer J401.13 (Pin_13)
- net TEST_CONN: now also J401.12 (Pin_12), U?.3 (IO2); no longer J401.2 (Pin_2)
Other:
- moved on the sheet: R412, R413, R414, R415, R416, R417, R?, U?

Commit message: Update PCB
Connections:
- net FL5_CONN: now also U?.1 (IO1); no longer U?.6 (IO4)
Changed lines of the file:
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@@
   (junction (at 143.51 85.09) (diameter 0) (color 0 0 0 0)
   )
+  (junction (at 190.5 77.47) (diameter 0) (color 0 0 0 0)
+  )
   (junction (at 160.02 82.55) (diameter 0) (color 0 0 0 0)
   )
-  (junction (at 179.07 77.47) (diameter 0) (color 0 0 0 0)
-  )
   (junction (at 163.83 74.93) (diameter 0) (color 0 0 0 0)
   )
@@
   (junction (at 138.43 87.63) (diameter 0) (color 0 0 0 0)
   )
-  (no_connect (at 190.5 99.06))
   (no_connect (at 163.83 99.06))
+  (no_connect (at 179.07 99.06))
   (wire (pts (xy 99.06 146.05) (xy 82.55 146.05))
     (stroke (width 0) (type default))
@@
     (stroke (width 0) (type default))
   )
+  (wire (pts (xy 190.5 77.47) (xy 190.5 99.06))
+    (stroke (width 0) (type default))
+  )
   (polyline (pts (xy 208.28 119.38) (xy 111.76 119.38))
     (stroke (width 0) (type default))
@@
     (stroke (width 0) (type default))
   )
-  (wire (pts (xy 158.75 77.47) (xy 179.07 77.47))
+  (wire (pts (xy 158.75 77.47) (xy 190.5 77.47))
     (stroke (width 0) (type default))
   )
@@
     (stroke (width 0) (type default))
   )
+  (wire (pts (xy 190.5 77.47) (xy 204.47 77.47))
+    (stroke (width 0) (type default))
+  )
   (wire (pts (xy 186.69 74.93) (xy 186.69 99.06))
     (stroke (width 0) (type default))
   )
-  (wire (pts (xy 179.07 77.47) (xy 179.07 99.06))
-    (stroke (width 0) (type default))
-  )
   (wire (pts (xy 82.55 151.13) (xy 85.09 151.13))
     (stroke (width 0) (type default))
@@
     (stroke (width 0) (type default))
   )
-  (wire (pts (xy 179.07 77.47) (xy 204.47 77.47))
-    (stroke (width 0) (type default))
-  )

Commit message: Update PCB
Parts:
- J401: value JST_B13P_XH -> JST_B13P_SHF_1AA
Other:
- moved on the sheet: J401, R401, R402, R403, R404, R405, R412, R413, R414, R415, R416, R417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

Commit message: Select input TVS diode
Other:
- title: BD845-PWB -> BD845-PWB SCH
Changed lines of the file:
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@@
   (paper "A4")
   (title_block
-    (title "BD845-PWB")
+    (title "BD845-PWB SCH")
     (date "2022-11-27")
-    (rev "1")
+    (rev "1.0.0")
     (company "BlueDot, Vincenzo Fortunato")
   )
