File: kicad/comm_channel.kicad_sch (KiCad schematic)
At the start: 25 parts, among them J401 JST_B13P_SHF_1AA, U401 EL357N(C)(TA)-G, U402 EL357N(C)(TA)-G, U403 EL357N(C)(TA)-G, U404 EL357N(C)(TA)-G, U405 EL357N(C)(TA)-G

Commit message: Update to v1.1.0
Parts:
- R401, R402, R403, R404, R405: JLCPCB Part # (none) -> C23138
- R412, R413, R414, R415, R416, R417: JLCPCB Part # (none) -> C25804
- R? (x6): JLCPCB Part # (none) -> C22808
- U401, U402, U403, U404, U405: JLCPCB Part # (none) -> C29981
- U? (x2): JLCPCB Part # (none) -> C85364
Other:
- company: BlueDot, Vincenzo Fortunato -> BlueDot Arcade, Vincenzo Fortunato
Changed lines of the file:
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@@
   (title_block
     (title "BD845-PWB SCH")
-    (date "2022-11-27")
-    (rev "1.0.0")
-    (company "BlueDot, Vincenzo Fortunato")
+    (date "2023-06-14")
+    (rev "1.1.0")
+    (company "BlueDot Arcade, Vincenzo Fortunato")
+    (comment 1 "bluedotarcade.com")
   )
   (junction (at 148.59 64.77) (diameter 0) (color 0 0 0 0)
@@
       (effects (font (size 1.27 1.27)) (justify left) hide)
     )
+    (property "JLCPCB Part #" "C29981" (at 69.85 129.54 0)
+      (effects (font (size 1.27 1.27)) hide)
+    )
     (pin "1")
     (pin "2")
@@
       (effects (font (size 1.27 1.27)) hide)
     )
+    (property "JLCPCB Part #" "C23138" (at 57.15 69.85 0)
+      (effects (font (size 1.27 1.27)) hide)
+    )
     (pin "1")
     (pin "2")
@@
       (effects (font (size 1.27 1.27)) hide)
     )
+    (property "JLCPCB Part #" "C23138" (at 57.15 88.9 0)
+      (effects (font (size 1.27 1.27)) hide)
+    )
     (pin "1")
     (pin "2")
@@
       (effects (font (size 1.27 1.27)) hide)
     )
+    (property "JLCPCB Part #" "C23138" (at 57.15 146.05 0)
+      (effects (font (size 1.27 1.27)) hide)
+    )
     (pin "1")
     (pin "2")
@@
       (effects (font (size 1.27 1.27)) hide)
     )
+    (property "JLCPCB Part #" "C23138" (at 57.15 107.95 0)
+      (effects (font (size 1.27 1.27)) hide)
+    )
     (pin "1")
     (pin "2")
@@
     )
     (property "Datasheet" "~" (at 255.27 87.63 0)
+      (effects (font (size 1.27 1.27)) hide)
+    )
+    (property "JLCPCB Part #" "" (at 255.27 87.63 0)
       (effects (font (size 1.27 1.27)) hide)
     )
@@
       (effects (font (size 1.27 1.27)) hide)
     )
+    (property "JLCPCB Part #" "C23138" (at 57.15 127 0)
+      (effects (font (size 1.27 1.27)) hide)
+    )
     (pin "1")
     (pin "2")
@@
     )
     (property "Datasheet" "~" (at 121.92 74.93 0)
+      (effects (font (size 1.27 1.27)) hide)
+    )
+    (property "JLCPCB Part #" "C22808" (at 121.92 74.93 0)
       (effects (font (size 1.27 1.27)) hide)
     )
@@
       (effects (font (size 1.27 1.27)) (justify left) hide)
     )
+    (property "JLCPCB Part #" "C29981" (at 69.85 148.59 0)
+      (effects (font (size 1.27 1.27)) hide)
+    )
     (pin "1")
     (pin "2")
@@
     )
     (property "Datasheet" "http://www.onsemi.com/pub/Collateral/SRV05-4-D.PDF" (at 175.26 86.36 0)
+      (effects (font (size 1.27 1.27)) hide)
+    )
+    (property "JLCPCB Part #" "C85364" (at 180.34 106.68 0)
       (effects (font (size 1.27 1.27)) hide)
     )
@@
       (effects (font (size 1.27 1.27)) hide)
     )
+    (property "JLCPCB Part #" "C22808" (at 121.92 80.01 0)
+      (effects (font (size 1.27 1.27)) hide)
+    )
     (pin "1")
     (pin "2")
@@
     )
     (property "Datasheet" "~" (at 153.67 68.58 0)
+      (effects (font (size 1.27 1.27)) hide)
+    )
+    (property "JLCPCB Part #" "C25804" (at 153.67 68.58 0)
       (effects (font (size 1.27 1.27)) hide)
     )
@@
     (property "Datasheet" "https://datasheet.lcsc.com/lcsc/1810271030_Everlight-Elec-EL357N-C-TA-G_C29981.pdf" (at 69.85 72.39 0)
       (effects (font (size 1.27 1.27)) (justify left) hide)
+    )
+    (property "JLCPCB Part #" "C29981" (at 69.85 72.39 0)
+      (effects (font (size 1.27 1.27)) hide)
     )
     (pin "1")
@@
       (effects (font (size 1.27 1.27)) hide)
     )
+    (property "JLCPCB Part #" "C22808" (at 121.92 87.63 0)
+      (effects (font (size 1.27 1.27)) hide)
+    )
     (pin "1")
     (pin "2")
@@
     )
     (property "Datasheet" "~" (at 148.59 68.58 0)
+      (effects (font (size 1.27 1.27)) hide)
+    )
+    (property "JLCPCB Part #" "C25804" (at 148.59 68.58 0)
       (effects (font (size 1.27 1.27)) hide)
     )
@@
       (effects (font (size 1.27 1.27)) (justify left) hide)
     )
+    (property "JLCPCB Part #" "C29981" (at 69.85 110.49 0)
+      (effects (font (size 1.27 1.27)) hide)
+    )
     (pin "1")
     (pin "2")
@@
     )
     (property "Datasheet" "http://www.onsemi.com/pub/Collateral/SRV05-4-D.PDF" (at 148.59 86.36 0)
+      (effects (font (size 1.27 1.27)) hide)
+    )
+    (property "JLCPCB Part #" "C85364" (at 153.67 106.68 0)
       (effects (font (size 1.27 1.27)) hide)
     )
@@
       (effects (font (size 1.27 1.27)) (justify left) hide)
     )
+    (property "JLCPCB Part #" "C29981" (at 69.85 91.44 0)
+      (effects (font (size 1.27 1.27)) hide)
+    )
     (pin "1")
     (pin "2")
@@
       (effects (font (size 1.27 1.27)) hide)
     )
+    (property "JLCPCB Part #" "C25804" (at 158.75 68.58 0)
+      (effects (font (size 1.27 1.27)) hide)
+    )
     (pin "1")
     (pin "2")
@@
       (effects (font (size 1.27 1.27)) hide)
     )
+    (property "JLCPCB Part #" "C25804" (at 133.35 68.58 0)
+      (effects (font (size 1.27 1.27)) hide)
+    )
     (pin "1")
     (pin "2")
@@
       (effects (font (size 1.27 1.27)) hide)
     )
+    (property "JLCPCB Part #" "C25804" (at 138.43 68.58 0)
+      (effects (font (size 1.27 1.27)) hide)
+    )
     (pin "1")
     (pin "2")
@@
       (effects (font (size 1.27 1.27)) hide)
     )
+    (property "JLCPCB Part #" "C22808" (at 121.92 77.47 0)
+      (effects (font (size 1.27 1.27)) hide)
+    )
     (pin "1")
     (pin "2")
@@
       (effects (font (size 1.27 1.27)) hide)
     )
+    (property "JLCPCB Part #" "C22808" (at 121.92 82.55 0)
+      (effects (font (size 1.27 1.27)) hide)
+    )
     (pin "1")
     (pin "2")
@@
       (effects (font (size 1.27 1.27)) hide)
     )
+    (property "JLCPCB Part #" "C22808" (at 121.92 85.09 0)
+      (effects (font (size 1.27 1.27)) hide)
+    )
     (pin "1")
     (pin "2")
@@
       (effects (font (size 1.27 1.27)) hide)
     )
+    (property "JLCPCB Part #" "C25804" (at 143.51 68.58 0)
+      (effects (font (size 1.27 1.27)) hide)
+    )
