File: kicad/comm_channel.kicad_sch (KiCad schematic)
At the start: 25 parts, among them J401 JST_B13P_SHF_1AA, U401 EL357N(C)(TA)-G, U402 EL357N(C)(TA)-G, U403 EL357N(C)(TA)-G, U404 EL357N(C)(TA)-G, U405 EL357N(C)(TA)-G

Commit message: fab: update BOM with missing component codes
Parts:
- J401: JLCPCB Part # (none) -> C160368
- U401, U402, U403, U404, U405: JLCPCB Part # C29981 -> C42432283
- gave numbers to parts that had none: 8
