File: kicad/mcu.kicad_sch (KiCad schematic)
At the start: 19 parts, among them J301 TC2030-MCP-NL, J302 PinHeader_01x05, U301 STM32F030C8Tx, U302 SRV05-4, Y301 16Mhz

Commit message: Update to v1.1.0
Parts:
- C301, C303: JLCPCB Part # (none) -> C1634
- C302, C305, C306, C307, C308: JLCPCB Part # (none) -> C14663
- C304: JLCPCB Part # (none) -> C96446
- R301: JLCPCB Part # (none) -> C25804
- R303: JLCPCB Part # (none) -> C23182
- R304, R305, R306: JLCPCB Part # (none) -> C22808
- U301: JLCPCB Part # (none) -> C23922
- U302: JLCPCB Part # (none) -> C85364
- Y301: JLCPCB Part # (none) -> C13738
Other:
- company: BlueDot, Vincenzo Fortunato -> BlueDot Arcade, Vincenzo Fortunato
Changed lines of the file:
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@@
   (title_block
     (title "BD845-PWB SCH")
-    (date "2022-11-27")
-    (rev "1.0.0")
-    (company "BlueDot, Vincenzo Fortunato")
+    (date "2023-06-14")
+    (rev "1.1.0")
+    (company "BlueDot Arcade, Vincenzo Fortunato")
+    (comment 1 "bluedotarcade.com")
   )
   (junction (at 109.22 55.88) (diameter 0) (color 0 0 0 0)
@@
       (effects (font (size 1.27 1.27)) hide)
     )
+    (property "JLCPCB Part #" "C14663" (at 82.55 48.26 0)
+      (effects (font (size 1.27 1.27)) hide)
+    )
     (pin "1")
     (pin "2")
@@
       (effects (font (size 1.27 1.27)) hide)
     )
+    (property "JLCPCB Part #" "C22808" (at 222.25 76.2 0)
+      (effects (font (size 1.27 1.27)) hide)
+    )
     (pin "1")
     (pin "2")
@@
     )
     (property "Datasheet" "~" (at 38.1 96.52 0)
+      (effects (font (size 1.27 1.27)) hide)
+    )
+    (property "JLCPCB Part #" "C1634" (at 38.1 96.52 0)
       (effects (font (size 1.27 1.27)) hide)
     )
@@
       (effects (font (size 1.27 1.27)) hide)
     )
+    (property "JLCPCB Part #" "C1634" (at 58.42 96.52 0)
+      (effects (font (size 1.27 1.27)) hide)
+    )
     (pin "1")
     (pin "2")
@@
       (effects (font (size 1.27 1.27)) hide)
     )
+    (property "JLCPCB Part #" "C22808" (at 222.25 72.39 0)
+      (effects (font (size 1.27 1.27)) hide)
+    )
     (pin "1")
     (pin "2")
@@
     )
     (property "Datasheet" "~" (at 45.72 58.42 0)
+      (effects (font (size 1.27 1.27)) hide)
+    )
+    (property "JLCPCB Part #" "C25804" (at 45.72 58.42 0)
       (effects (font (size 1.27 1.27)) hide)
     )
@@
     )
     (property "Datasheet" "~" (at 55.88 66.04 0)
+      (effects (font (size 1.27 1.27)) hide)
+    )
+    (property "JLCPCB Part #" "C14663" (at 55.88 66.04 0)
       (effects (font (size 1.27 1.27)) hide)
     )
@@
       (effects (font (size 1.27 1.27)) hide)
     )
+    (property "JLCPCB Part #" "C85364" (at 201.93 95.25 0)
+      (effects (font (size 1.27 1.27)) hide)
+    )
     (pin "1")
     (pin "2")
@@
     )
     (property "Datasheet" "http://www.st.com/st-web-ui/static/active/en/resource/technical/document/datasheet/DM00088500.pdf" (at 105.41 107.95 0)
+      (effects (font (size 1.27 1.27)) hide)
+    )
+    (property "JLCPCB Part #" "C23922" (at 105.41 107.95 0)
       (effects (font (size 1.27 1.27)) hide)
     )
@@
       (effects (font (size 1.27 1.27)) hide)
     )
+    (property "JLCPCB Part #" "C14663" (at 73.66 48.26 0)
+      (effects (font (size 1.27 1.27)) hide)
+    )
     (pin "1")
     (pin "2")
@@
     )
     (property "Datasheet" "~" (at 48.26 92.71 0)
+      (effects (font (size 1.27 1.27)) hide)
+    )
+    (property "JLCPCB Part #" "C13738" (at 48.26 92.71 0)
       (effects (font (size 1.27 1.27)) hide)
     )
@@
       (effects (font (size 1.27 1.27)) hide)
     )
+    (property "JLCPCB Part #" "C14663" (at 91.44 48.26 0)
+      (effects (font (size 1.27 1.27)) hide)
+    )
     (pin "1")
     (pin "2")
@@
     )
     (property "Datasheet" "~" (at 100.33 48.26 0)
+      (effects (font (size 1.27 1.27)) hide)
+    )
+    (property "JLCPCB Part #" "C14663" (at 100.33 48.26 0)
       (effects (font (size 1.27 1.27)) hide)
     )
@@
     )
     (property "Datasheet" "~" (at 223.52 52.07 0)
+      (effects (font (size 1.27 1.27)) hide)
+    )
+    (property "JLCPCB Part #" "" (at 223.52 52.07 0)
       (effects (font (size 1.27 1.27)) hide)
     )
@@
       (effects (font (size 1.27 1.27)) hide)
     )
+    (property "JLCPCB Part #" "C96446" (at 64.77 48.26 0)
+      (effects (font (size 1.27 1.27)) hide)
+    )
     (pin "1")
     (pin "2")
@@
       (effects (font (size 1.27 1.27)) hide)
     )
+    (property "JLCPCB Part #" "C22808" (at 222.25 80.01 0)
+      (effects (font (size 1.27 1.27)) hide)
+    )
     (pin "1")
     (pin "2")
@@
     (property "Arrow Price/Stock" "https://www.arrow.com/en/products/tc2030-mcp-nl/microchip-technology?region=nac" (at 162.56 72.39 0)
       (effects (font (size 1.27 1.27)) (justify left) hide)
+    )
+    (property "JLCPCB Part #" "" (at 191.77 53.34 0)
+      (effects (font (size 1.27 1.27)) hide)
     )
     (pin "1")
@@
       (effects (font (size 1.27 1.27)) hide)
     )
+    (property "JLCPCB Part #" "" (at 45.72 66.04 0)
+      (effects (font (size 1.27 1.27)) hide)
+    )
     (pin "1")
     (pin "2")
@@
       (effects (font (size 1.27 1.27)) hide)
     )
+    (property "JLCPCB Part #" "C23182" (at 58.42 88.9 0)
+      (effects (font (size 1.27 1.27)) hide)
+    )
