File: kicad/bd845-pwb.kicad_sch (KiCad schematic)
At the start: 27 parts, among them J101 JST_VH_B4P, SW101 SW_DIP_x04, U101 74HC595, U102 74HC595

Commit message: Update to v1.1.0
Parts:
- C101, C102, C103, C104: JLCPCB Part # (none) -> C1588
- C105, C108: JLCPCB Part # (none) -> C57112
- C106, C107: JLCPCB Part # (none) -> C14663
- D101: JLCPCB Part # (none) -> C2296
- R101: JLCPCB Part # (none) -> C23138
- R? (x4): JLCPCB Part # (none) -> C22808
- R? (x4): JLCPCB Part # (none) -> C25804
- SW101: JLCPCB Part # (none) -> C692502
- U101, U102: JLCPCB Part # (none) -> C5947
- U?: JLCPCB Part # (none) -> C85364
Other:
- company: BlueDot, Vincenzo Fortunato -> BlueDot Arcade, Vincenzo Fortunato
Changed lines of the file:
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@@
   (title_block
     (title "BD845-PWB SCH")
-    (date "2022-11-27")
-    (rev "1.0.0")
-    (company "BlueDot, Vincenzo Fortunato")
+    (date "2023-06-14")
+    (rev "1.1.0")
+    (company "BlueDot Arcade, Vincenzo Fortunato")
+    (comment 1 "bluedotarcade.com")
   )
   (junction (at 276.86 127) (diameter 0) (color 0 0 0 0)
@@
       (effects (font (size 1.27 1.27)) hide)
     )
+    (property "JLCPCB Part #" "C57112" (at 240.03 55.88 0)
+      (effects (font (size 1.27 1.27)) hide)
+    )
     (pin "1")
     (pin "2")
@@
       (effects (font (size 1.27 1.27)) hide)
     )
+    (property "JLCPCB Part #" "" (at 100.33 162.56 0)
+      (effects (font (size 1.27 1.27)) hide)
+    )
     (pin "1")
     (instances
@@
       (effects (font (size 1.27 1.27)) hide)
     )
+    (property "JLCPCB Part #" "C1588" (at 93.98 168.91 0)
+      (effects (font (size 1.27 1.27)) hide)
+    )
     (pin "1")
     (pin "2")
@@
     )
     (property "Datasheet" "~" (at 212.09 129.54 0)
+      (effects (font (size 1.27 1.27)) hide)
+    )
+    (property "JLCPCB Part #" "C22808" (at 212.09 129.54 0)
       (effects (font (size 1.27 1.27)) hide)
     )
@@
       (effects (font (size 1.27 1.27)) hide)
     )
+    (property "JLCPCB Part #" "C1588" (at 93.98 175.26 0)
+      (effects (font (size 1.27 1.27)) hide)
+    )
     (pin "1")
     (pin "2")
@@
     )
     (property "Datasheet" "~" (at 212.09 124.46 0)
+      (effects (font (size 1.27 1.27)) hide)
+    )
+    (property "JLCPCB Part #" "C22808" (at 212.09 124.46 0)
       (effects (font (size 1.27 1.27)) hide)
     )
@@
       (effects (font (size 1.27 1.27)) hide)
     )
+    (property "JLCPCB Part #" "C25804" (at 224.79 133.35 0)
+      (effects (font (size 1.27 1.27)) hide)
+    )
     (pin "1")
     (pin "2")
@@
     )
     (property "Datasheet" "~" (at 240.03 133.35 0)
+      (effects (font (size 1.27 1.27)) hide)
+    )
+    (property "JLCPCB Part #" "C25804" (at 240.03 133.35 0)
       (effects (font (size 1.27 1.27)) hide)
     )
@@
       (effects (font (size 1.27 1.27)) hide)
     )
+    (property "JLCPCB Part #" "C25804" (at 234.95 133.35 0)
+      (effects (font (size 1.27 1.27)) hide)
+    )
     (pin "1")
     (pin "2")
@@
       (effects (font (size 1.27 1.27)) hide)
     )
+    (property "JLCPCB Part #" "C1588" (at 93.98 162.56 0)
+      (effects (font (size 1.27 1.27)) hide)
+    )
     (pin "1")
     (pin "2")
@@
       (effects (font (size 1.27 1.27)) hide)
     )
+    (property "JLCPCB Part #" "" (at 100.33 168.91 0)
+      (effects (font (size 1.27 1.27)) hide)
+    )
     (pin "1")
     (instances
@@
     )
     (property "Datasheet" "~" (at 100.33 175.26 0)
+      (effects (font (size 1.27 1.27)) hide)
+    )
+    (property "JLCPCB Part #" "" (at 100.33 175.26 0)
       (effects (font (size 1.27 1.27)) hide)
     )
@@
       (effects (font (size 1.27 1.27)) hide)
     )
+    (property "JLCPCB Part #" "C14663" (at 229.87 55.88 0)
+      (effects (font (size 1.27 1.27)) hide)
+    )
     (pin "1")
     (pin "2")
@@
       (effects (font (size 1.27 1.27)) hide)
     )
+    (property "JLCPCB Part #" "C14663" (at 106.68 90.17 0)
+      (effects (font (size 1.27 1.27)) hide)
+    )
     (pin "1")
     (pin "2")
@@
     )
     (property "Datasheet" "~" (at 100.33 156.21 0)
+      (effects (font (size 1.27 1.27)) hide)
+    )
+    (property "JLCPCB Part #" "" (at 100.33 156.21 0)
       (effects (font (size 1.27 1.27)) hide)
     )
@@
       (effects (font (size 1.27 1.27)) hide)
     )
+    (property "JLCPCB Part #" "C57112" (at 96.52 90.17 0)
+      (effects (font (size 1.27 1.27)) hide)
+    )
     (pin "1")
     (pin "2")
@@
     )
     (property "Datasheet" "http://www.ti.com/lit/ds/symlink/sn74hc595.pdf" (at 219.71 80.01 0)
+      (effects (font (size 1.27 1.27)) hide)
+    )
+    (property "JLCPCB Part #" "C5947" (at 219.71 80.01 0)
       (effects (font (size 1.27 1.27)) hide)
     )
@@
       (effects (font (size 1.27 1.27)) hide)
     )
+    (property "JLCPCB Part #" "C23138" (at 162.56 143.51 0)
+      (effects (font (size 1.27 1.27)) hide)
+    )
     (pin "1")
     (pin "2")
@@
     )
     (property "Datasheet" "~" (at 266.7 124.46 0)
+      (effects (font (size 1.27 1.27)) hide)
+    )
+    (property "JLCPCB Part #" "C692502" (at 266.7 124.46 0)
       (effects (font (size 1.27 1.27)) hide)
     )
@@
       (effects (font (size 1.27 1.27)) hide)
     )
+    (property "JLCPCB Part #" "C2296" (at 142.24 143.51 0)
+      (effects (font (size 1.27 1.27)) hide)
+    )
     (pin "1")
     (pin "2")
@@
     )
     (property "Datasheet" "~" (at 229.87 133.35 0)
+      (effects (font (size 1.27 1.27)) hide)
+    )
+    (property "JLCPCB Part #" "C25804" (at 229.87 133.35 0)
       (effects (font (size 1.27 1.27)) hide)
     )
@@
     )
     (property "Datasheet" "http://www.onsemi.com/pub/Collateral/SRV05-4-D.PDF" (at 255.27 127 0)
+      (effects (font (size 1.27 1.27)) hide)
+    )
+    (property "JLCPCB Part #" "C85364" (at 250.19 147.32 0)
       (effects (font (size 1.27 1.27)) hide)
     )
@@
       (effects (font (size 1.27 1.27)) hide)
     )
+    (property "JLCPCB Part #" "C1588" (at 93.98 156.21 0)
+      (effects (font (size 1.27 1.27)) hide)
+    )
     (pin "1")
     (pin "2")
@@
     )
     (property "Datasheet" "http://www.ti.com/lit/ds/symlink/sn74hc595.pdf" (at 116.84 114.3 0)
+      (effects (font (size 1.27 1.27)) hide)
+    )
+    (property "JLCPCB Part #" "C5947" (at 116.84 114.3 0)
       (effects (font (size 1.27 1.27)) hide)
     )
@@
       (effects (font (size 1.27 1.27)) hide)
     )
+    (property "JLCPCB Part #" "C22808" (at 212.09 127 0)
+      (effects (font (size 1.27 1.27)) hide)
+    )
     (pin "1")
     (pin "2")
@@
     )
     (property "Datasheet" "~" (at 125.73 176.53 0)
+      (effects (font (size 1.27 1.27)) hide)
+    )
+    (property "JLCPCB Part #" "" (at 125.73 176.53 0)
       (effects (font (size 1.27 1.27)) hide)
     )
@@
       (effects (font (size 1.27 1.27)) hide)
     )
+    (property "JLCPCB Part #" "C22808" (at 212.09 121.92 0)
+      (effects (font (size 1.27 1.27)) hide)
+    )

Commit message: Change light driver to a self-protected mosfet. Remove unnecessary fuses. Change 74HC595 to low input voltage equivalent. Change LED resistors to 1k. Power lights shift register with +5V.
Parts:
- R101: value 330R -> 1k; JLCPCB Part # C23138 -> C21190
- U101: value 74HC595 -> 74HC595-Q100; JLCPCB Part # C5947 -> C547127
- U102: JLCPCB Part # C5947 -> C547127
Connections:
- net +3V3: no longer C105.1, C106.1, U101.10 (~{SRCLR}), U101.16 (VCC)
- new net +5V: C105.1, C106.1, U101.10 (~{SRCLR}), U101.16 (VCC)
- no-connect marks 8 -> 7
Changed lines of the file:
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@@
   (junction (at 86.36 162.56) (diameter 0) (color 0 0 0 0)
   )
+  (junction (at 154.94 162.56) (diameter 0) (color 0 0 0 0)
+  )
   (junction (at 224.79 137.16) (diameter 0) (color 0 0 0 0)
   )
@@
   (junction (at 229.87 124.46) (diameter 0) (color 0 0 0 0)
   )
+  (junction (at 161.29 162.56) (diameter 0) (color 0 0 0 0)
+  )
   (junction (at 224.79 121.92) (diameter 0) (color 0 0 0 0)
   )
@@
   (junction (at 96.52 93.98) (diameter 0) (color 0 0 0 0)
   )
+  (junction (at 167.64 162.56) (diameter 0) (color 0 0 0 0)
+  )
   (junction (at 229.87 137.16) (diameter 0) (color 0 0 0 0)
   )
@@
   (junction (at 240.03 59.69) (diameter 0) (color 0 0 0 0)
   )
-  (no_connect (at 161.29 161.29))
   (no_connect (at 106.68 121.92))
   (no_connect (at 229.87 87.63))
@@
     (stroke (width 0) (type default))
   )
+  (wire (pts (xy 161.29 162.56) (xy 161.29 165.1))
+    (stroke (width 0) (type default))
+  )
   (wire (pts (xy 201.93 77.47) (xy 201.93 82.55))
     (stroke (width 0) (type default))
@@
     (stroke (width 0) (type default))
   )
-  (wire (pts (xy 167.64 161.29) (xy 167.64 165.1))
+  (wire (pts (xy 167.64 161.29) (xy 167.64 162.56))
     (stroke (width 0) (type default))
   )
@@
     (stroke (width 0) (type default))
   )
-  (wire (pts (xy 154.94 161.29) (xy 154.94 165.1))
+  (wire (pts (xy 154.94 161.29) (xy 154.94 162.56))
+    (stroke (width 0) (type default))
+  )
+  (wire (pts (xy 154.94 162.56) (xy 154.94 165.1))
     (stroke (width 0) (type default))
   )
@@
     (stroke (width 0) (type default))
   )
+  (wire (pts (xy 167.64 162.56) (xy 167.64 165.1))
+    (stroke (width 0) (type default))
+  )
   (bus (pts (xy 134.62 67.31) (xy 134.62 69.85))
     (stroke (width 0) (type default))
@@
     (stroke (width 0) (type default))
   )
-  (wire (pts (xy 161.29 161.29) (xy 161.29 165.1))
+  (wire (pts (xy 161.29 161.29) (xy 161.29 162.56))
     (stroke (width 0) (type default))
   )
@@
     )
   )
+  (symbol (lib_id "power:+5V") (at 161.29 161.29 0) (unit 1)
+    (in_bom yes) (on_board yes) (dnp no)
+    (property "Reference" "#PWR02" (at 161.29 165.1 0)
+      (effects (font (size 1.27 1.27)) hide)
+    )
+    (property "Value" "+5V" (at 161.29 157.48 0)
+      (effects (font (size 1.27 1.27)))
+    )
+    (property "Footprint" "" (at 161.29 161.29 0)
+      (effects (font (size 1.27 1.27)) hide)
+    )
+    (property "Datasheet" "" (at 161.29 161.29 0)
+      (effects (font (size 1.27 1.27)) hide)
+    )
+    (pin "1")
+    (instances
+      (project "bd845-pwb"
+        (path "/c0443f53-6229-4858-b0f1-180b8ed8e6c2"
+          (reference "#PWR02") (unit 1)
+        )
+      )
+    )
+  )
   (symbol (lib_id "Device:R_Small") (at 212.09 129.54 270) (unit 1)
     (in_bom yes) (on_board yes) (dnp no)
@@
     )
   )
+  (symbol (lib_id "power:+5V") (at 129.54 101.6 0) (unit 1)
+    (in_bom yes) (on_board yes) (dnp no)
+    (property "Reference" "#PWR03" (at 129.54 105.41 0)
+      (effects (font (size 1.27 1.27)) hide)
+    )
+    (property "Value" "+5V" (at 129.54 97.79 0)
+      (effects (font (size 1.27 1.27)))
+    )
+    (property "Footprint" "" (at 129.54 101.6 0)
+      (effects (font (size 1.27 1.27)) hide)
+    )
+    (property "Datasheet" "" (at 129.54 101.6 0)
+      (effects (font (size 1.27 1.27)) hide)
+    )
+    (pin "1")
+    (instances
+      (project "bd845-pwb"
+        (path "/c0443f53-6229-4858-b0f1-180b8ed8e6c2"
+          (reference "#PWR03") (unit 1)
+        )
+      )
+    )
+  )
   (symbol (lib_id "Device:R_Small") (at 240.03 133.35 0) (mirror y) (unit 1)
     (in_bom yes) (on_board yes) (dnp no)
@@
         (path "/c0443f53-6229-4858-b0f1-180b8ed8e6c2"
           (reference "#PWR0119") (unit 1)
-        )
-      )
-    )
-  )
-  (symbol (lib_id "power:+3V3") (at 129.54 101.6 0) (unit 1)
-    (in_bom yes) (on_board yes) (dnp no) (fields_autoplaced)
-    (property "Reference" "#PWR0117" (at 129.54 105.41 0)
-      (effects (font (size 1.27 1.27)) hide)
-    )
-    (property "Value" "+3V3" (at 129.54 97.79 0)
-      (effects (font (size 1.27 1.27)))
-    )
-    (property "Footprint" "" (at 129.54 101.6 0)
-      (effects (font (size 1.27 1.27)) hide)
-    )
-    (property "Datasheet" "" (at 129.54 101.6 0)
-      (effects (font (size 1.27 1.27)) hide)
-    )
-    (pin "1")
-    (instances
-      (project "bd845-pwb"
-        (path "/c0443f53-6229-4858-b0f1-180b8ed8e6c2"
-          (reference "#PWR0117") (unit 1)
         )
       )
@@
     )
   )
+  (symbol (lib_id "power:PWR_FLAG") (at 167.64 162.56 90) (unit 1)
+    (in_bom yes) (on_board yes) (dnp no) (fields_autoplaced)
+    (property "Reference" "#FLG03" (at 165.735 162.56 0)
+      (effects (font (size 1.27 1.27)) hide)
+    )
+    (property "Value" "PWR_FLAG" (at 163.83 162.56 90)
+      (effects (font (size 1.27 1.27)) (justify left) hide)
+    )
+    (property "Footprint" "" (at 167.64 162.56 0)
+      (effects (font (size 1.27 1.27)) hide)
+    )
+    (property "Datasheet" "~" (at 167.64 162.56 0)
+      (effects (font (size 1.27 1.27)) hide)
+    )
+    (pin "1")
+    (instances
+      (project "bd845-pwb"
+        (path "/c0443f53-6229-4858-b0f1-180b8ed8e6c2"
+          (reference "#FLG03") (unit 1)
+        )
+      )
+    )
+  )
   (symbol (lib_id "power:GND") (at 129.54 121.92 0) (unit 1)
     (in_bom yes) (on_board yes) (dnp no)
@@
       (effects (font (size 1.27 1.27)) hide)
     )
-    (property "JLCPCB Part #" "C5947" (at 219.71 80.01 0)
+    (property "JLCPCB Part #" "C547127" (at 219.71 80.01 0)
       (effects (font (size 1.27 1.27)) hide)
     )
@@
       (effects (font (size 1.27 1.27)))
     )
-    (property "Value" "330R" (at 162.56 146.05 90)
+    (property "Value" "1k" (at 162.56 146.05 90)
       (effects (font (size 1.27 1.27)))
     )
@@
       (effects (font (size 1.27 1.27)) hide)
     )
-    (property "JLCPCB Part #" "C23138" (at 162.56 143.51 0)
+    (property "JLCPCB Part #" "C21190" (at 162.56 143.51 0)
       (effects (font (size 1.27 1.27)) hide)
     )
@@
     )
   )
-  (symbol (lib_id "power:+3V3") (at 116.84 85.09 0) (mirror y) (unit 1)
-    (in_bom yes) (on_board yes) (dnp no) (fields_autoplaced)
-    (property "Reference" "#PWR0115" (at 116.84 88.9 0)
-      (effects (font (size 1.27 1.27)) hide)
-    )
-    (property "Value" "+3V3" (at 116.84 81.28 0)
-      (effects (font (size 1.27 1.27)))
-    )
-    (property "Footprint" "" (at 116.84 85.09 0)
-      (effects (font (size 1.27 1.27)) hide)
-    )
-    (property "Datasheet" "" (at 116.84 85.09 0)
-      (effects (font (size 1.27 1.27)) hide)
-    )
-    (pin "1")
-    (instances
-      (project "bd845-pwb"
-        (path "/c0443f53-6229-4858-b0f1-180b8ed8e6c2"
-          (reference "#PWR0115") (unit 1)
-        )
-      )
-    )
-  )
   (symbol (lib_id "ProjectLibrary:SRV05-4") (at 250.19 147.32 0) (unit 1)
     (in_bom yes) (on_board yes) (dnp no)
@@
     )
   )
+  (symbol (lib_id "power:PWR_FLAG") (at 161.29 162.56 90) (unit 1)
+    (in_bom yes) (on_board yes) (dnp no) (fields_autoplaced)
+    (property "Reference" "#FLG02" (at 159.385 162.56 0)
+      (effects (font (size 1.27 1.27)) hide)
+    )
+    (property "Value" "PWR_FLAG" (at 157.48 162.56 90)
+      (effects (font (size 1.27 1.27)) (justify left) hide)
+    )
+    (property "Footprint" "" (at 161.29 162.56 0)
+      (effects (font (size 1.27 1.27)) hide)
+    )
+    (property "Datasheet" "~" (at 161.29 162.56 0)
+      (effects (font (size 1.27 1.27)) hide)
+    )
+    (pin "1")
+    (instances
+      (project "bd845-pwb"
+        (path "/c0443f53-6229-4858-b0f1-180b8ed8e6c2"
+          (reference "#FLG02") (unit 1)
+        )
+      )
+    )
+  )
   (symbol (lib_id "Device:C_Small") (at 93.98 156.21 90) (unit 1)
     (in_bom yes) (on_board yes) (dnp no)
@@
     )
   )
+  (symbol (lib_id "power:PWR_FLAG") (at 154.94 162.56 90) (unit 1)
+    (in_bom yes) (on_board yes) (dnp no)
+    (property "Reference" "#FLG01" (at 153.035 162.56 0)
+      (effects (font (size 1.27 1.27)) hide)
+    )
+    (property "Value" "PWR_FLAG" (at 179.07 162.56 90)
+      (effects (font (size 1.27 1.27)) (justify left))
+    )
+    (property "Footprint" "" (at 154.94 162.56 0)
+      (effects (font (size 1.27 1.27)) hide)
+    )
+    (property "Datasheet" "~" (at 154.94 162.56 0)
+      (effects (font (size 1.27 1.27)) hide)
+    )
+    (pin "1")
+    (instances
+      (project "bd845-pwb"
+        (path "/c0443f53-6229-4858-b0f1-180b8ed8e6c2"
+          (reference "#FLG01") (unit 1)
+        )
+      )
+    )
+  )
   (symbol (lib_id "74xx:74HC595") (at 116.84 114.3 0) (mirror y) (unit 1)
     (in_bom yes) (on_board yes) (dnp no)
-    (property "Reference" "U101" (at 113.03 96.52 0)
+    (property "Reference" "U101" (at 115.57 95.25 0)
       (effects (font (size 1.27 1.27)) (justify left))
     )
-    (property "Value" "74HC595" (at 113.03 99.06 0)
+    (property "Value" "74HC595-Q100" (at 115.57 97.79 0)
       (effects (font (size 1.27 1.27)) (justify left))
     )
@@
       (effects (font (size 1.27 1.27)) hide)
     )
-    (property "JLCPCB Part #" "C5947" (at 116.84 114.3 0)
+    (property "JLCPCB Part #" "C547127" (at 116.84 114.3 0)
       (effects (font (size 1.27 1.27)) hide)
     )
@@
         )
       )
+    )
+  )
+  (symbol (lib_id "power:+5V") (at 116.84 85.09 0) (unit 1)
+    (in_bom yes) (on_board yes) (dnp no)
+    (property "Reference" "#PWR01" (at 116.84 88.9 0)
+      (effects (font (size 1.27 1.27)) hide)
+    )
+    (property "Value" "+5V" (at 116.84 81.28 0)
+      (effects (font (size 1.27 1.27)))
+    )
+    (property "Footprint" "" (at 116.84 85.09 0)
+      (effects (font (size 1.27 1.27)) hide)
+    )
+    (property "Datasheet" "" (at 116.84 85.09 0)
+      (effects (font (size 1.27 1.27)) hide)
+    )
+    (pin "1")
+    (instances
+      (project "bd845-pwb"
+        (path "/c0443f53-6229-4858-b0f1-180b8ed8e6c2"
+          (reference "#PWR01") (unit 1)
+        )
+      )
