File: kicad/bd845-pwb.kicad_sch (KiCad schematic)
At the start: 27 parts, among them J101 JST_VH_B4P, SW101 SW_DIP_x04, U101 74HC595-Q100, U102 74HC595

Commit message: fab: update BOM with missing component codes
Parts:
- J101: JLCPCB Part # (none) -> C493148
- U101, U102: JLCPCB Part # C547127 -> C5947
- gave numbers to parts that had none: 9
