File: kicad/pad_channel.kicad_sch (KiCad schematic)
At the start: 14 parts, among them J501 JST_B11P_SHF_1AA, Q501 ZXMS6004FFTA, U501 SRV05-4

Commit message: fab: update BOM with missing component codes
Parts:
- J501: JLCPCB Part # (none) -> C160366
