File: kicad/power.kicad_sch (KiCad schematic)
At the start: 39 parts, among them Q201 AOD409, U201 AMS1117-3.3, U202 TPS54331

Commit message: fab: update BOM with missing component codes
Parts:
- D201: JLCPCB Part # C110044 -> C19077536
- D202: JLCPCB Part # C8062 -> C19077402
- D203: JLCPCB Part # C142303 -> C2297
- renumbered R101 to R202
